File: H12R00/Design/H12R00.sch (EAGLE design)
At the start: 35 parts, among them P1 HEXABIT_17.32_NO_P3_P6, U1 STM32F091CBU6, U2 AD628ARZ, U3 REF193GSZ, X1 XTALL_CSTCE8M00G52

Commit message: - Fixed C11 and C14 attributes..
Parts:
- C11, C14: DESCREPTION Ceramic capacitor SMD-1206 100nF /50V X7R# K +-10%, AVX, Ro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 -> CAP CER 10% X7R 0603; MFN AVX -> KEMET; MPN 12065C104KAT2A -> C0603C104K8RACTU; OCTOPART_URL https://octopart.com/12065c104kat2a-avx-39590617 -> https://octopart.com/c0603c103k5ractu-kemet-133094?r=sp&s=R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
Changed lines of the file:
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@@
 <?xml version="1.0" encoding="utf-8"?>
 <!DOCTYPE eagle SYSTEM "eagle.dtd">
-<eagle version="9.3.0">
+<eagle version="9.6.2">
 <drawing>
 <settings>
-<setting alwaysvectorfont="yes"/>
+<setting alwaysvectorfont="no"/>
 <setting verticaltext="up"/>
 </settings>
@@
 <attribute name="CAPACITANCE" value="100 nF"/>
 <attribute name="CAPACITANCE_TOLERANCE" value="±10%"/>
-<attribute name="DESCREPTION" value="Ceramic capacitor SMD-1206 100nF /50V X7R# K +-10%, AVX, RoHS, /4000 reel/"/>
-<attribute name="MFN" value="AVX"/>
-<attribute name="MPN" value="12065C104KAT2A"/>
-<attribute name="OCTOPART_URL" value="https://octopart.com/12065c104kat2a-avx-39590617"/>
+<attribute name="DESCREPTION" value="CAP CER  10% X7R 0603"/>
+<attribute name="MFN" value="KEMET"/>
+<attribute name="MPN" value="C0603C104K8RACTU"/>
+<attribute name="OCTOPART_URL" value="https://octopart.com/c0603c103k5ractu-kemet-133094?r=sp&amp;s=R_iPBxLnSmGqhkU2rIMFpg"/>
 <attribute name="VOLTAGE_RATING" value="50.0 V"/>
 </part>
@@
 <attribute name="CAPACITANCE" value="100 nF"/>
 <attribute name="CAPACITANCE_TOLERANCE" value="±10%"/>
-<attribute name="DESCREPTION" value="Ceramic capacitor SMD-1206 100nF /50V X7R# K +-10%, AVX, RoHS, /4000 reel/"/>
-<attribute name="MFN" value="AVX"/>
-<attribute name="MPN" value="12065C104KAT2A"/>
-<attribute name="OCTOPART_URL" value="https://octopart.com/12065c104kat2a-avx-39590617"/>
+<attribute name="DESCREPTION" value="CAP CER  10% X7R 0603"/>
+<attribute name="MFN" value="KEMET"/>
+<attribute name="MPN" value="C0603C104K8RACTU"/>
+<attribute name="OCTOPART_URL" value="https://octopart.com/c0603c103k5ractu-kemet-133094?r=sp&amp;s=R_iPBxLnSmGqhkU2rIMFpg"/>
 <attribute name="VOLTAGE_RATING" value="50.0 V"/>
 </part>

Commit message: - Fixed labels in .sch and .brd from 12v to 10v - Regenerated docoument file - Fixed BOM - Regenerated output files (Gerber, drills, mount)
Other:
- note added: "Analog Input (0-10v)"
- note added: "Industrial 12-Bit (0-10v) Analog Input Module"
- note removed: "Analog Input (0-12v)"
- note removed: "Industrial 12-Bit (0-12v) Analog Input Module"
Changed lines of the file:
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@@
 <text x="199.4662" y="19.6342" size="1.9304" layer="100" font="vector">Title</text>
 <text x="180.9242" y="19.6342" size="1.9304" layer="102" font="vector">H12R00</text>
-<text x="193.2178" y="11.8364" size="1.9304" layer="101" font="vector" align="center">Industrial 12-Bit (0-12v)
+<text x="193.2178" y="11.8364" size="1.9304" layer="101" font="vector" align="center">Industrial 12-Bit (0-10v)
 Analog Input Module</text>
 <text x="206.3242" y="19.6342" size="1.9304" layer="101" font="vector">H12R00_Backend</text>
@@
 <text x="199.4662" y="19.6342" size="1.9304" layer="100" font="vector">Title</text>
 <text x="180.9242" y="19.6342" size="1.9304" layer="102" font="vector">H12R00</text>
-<text x="191.9478" y="11.9634" size="1.9304" layer="101" font="vector" align="center">Industrial 12-Bit (0-12v)
+<text x="191.9478" y="11.9634" size="1.9304" layer="101" font="vector" align="center">Industrial 12-Bit (0-10v)
 Analog Input Module</text>
 <text x="206.3242" y="19.6342" size="1.9304" layer="101" font="vector">H12R00_Frontend</text>
@@
 <text x="21.209" y="194.437" size="2.1844" layer="150">VDD = 3.3v</text>
 <text x="180.1622" y="4.9022" size="1.9304" layer="102" font="vector">Anas Kaadan</text>
-<text x="253.619" y="165.227" size="2.1844" layer="150" rot="R180">Analog Input (0-12v)</text>
+<text x="253.619" y="165.227" size="2.1844" layer="150" rot="R180">Analog Input (0-10v)</text>
 <text x="19.939" y="158.877" size="2.1844" layer="150">+15v</text>
 <text x="22.479" y="146.177" size="2.1844" layer="150">0v</text>

Commit message: - Made some Hardware modifications (.sch and .brd where updated) - Updated Documentation - Updated BOM - Regenerated output files
Parts:
- removed C14: 100 nF, Hexabitz:C-1206
- removed U3: REF193GSZ, Hexabitz:REF193GSZANALOG_DEVICES_REF193GSZ_0_1
- added R4: 62k, HEXABITZ_RCLS:R-0402
- added TVS2, TVS3: SMBJ3V3, HEXABITZ_RCLS:SMBJ3V3
- R5: value 10 kΩ -> 51 kΩ; device Hexabitz:R-0805 -> HEXABITZ_RCLS:R-0402; MFN Vishay -> Panasonic; MPN CRCW080510K0FKEA -> ERJ-2RKF5102X; OCTOPART_URL https://octopart.com/crcw080510k0fkea-vishay-39436722 -> https://octopart.com/erj-2rkf5102x-panasonic-42799737?r=sp; RESISTANCE 10 kΩ -> 51 kΩ
- R6: value 15 kΩ -> 22 kΩ; device Hexabitz:R-0805 -> HEXABITZ_RCLS:R-0603; MFN Vishay -> Yageo; MPN CRCW080515K0FKEA -> RT0603FRE0722KL; OCTOPART_URL https://octopart.com/crcw080515k0fkea-vishay-39456030 -> https://octopart.com/rt0603fre0722kl-yageo-40031569?r=sp; RESISTANCE 15 KΩ -> 22 KΩ
Connections:
- removed net 3V0: C1.1, C14.1, C2.+, U1.VDDA, U3.OUTPUT
- removed net UART6_RX: U1.PA5
- removed net UART6_TX: U1.PA4
- new net AGND: TVS2.1, TVS3.1
- new net VOLTAGE_SCALE: R4.1, TVS2.2, U1.PB1
- net +15V: now also R4.2; no longer U3.!SLEEP!, U3.VS
- net GND: now also U1.PA4
- net N$1: now also TVS3.2
- net VDD: now also C1.1, C2.+, U1.VDDA
- net VSSA: no longer C14.2, U3.GND
Other:
- note added: "12/15v"
- note added: "12v -> Voltage scale = 2.8v"
- note added: "15v -> Voltage scale = 3.3v"
- note removed: "+15v"
- moved on the sheet: C12, R7
