File: H12R00/Design/H12R00.sch (EAGLE design)
At the start: 42 parts, among them J1 1984646, P1 HEXABIT_17.32_NO_P6_P7_P12, U1 STM32G0B1CEU6N, U2 AD628ARZ, U3 TEXAS_INSTRUMENTS_REF2033AIDD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, X1 XTALL_CSTCE8M00G52

Commit message: -After wiring
Parts:
- X1: device Hexabitz:XTALL_CSTCE8M00G52 -> HEXABITZ_RCLS:XTALL_CSTCE8M00G52
Connections:
- removed net N$15: R2.1, U1.PB14
- removed net USART6_RX: U1.PA5
- removed net USART6_TX: U1.PA4
- new net N$4: R2.1, U1.PB2
- new net USART3_RX: P1.SD3, U1.PB11
- new net USART3_TX: P1.SU3, U1.PB10
- net GND: now also U1.PA9
- net M_SIG: now also U1.PA4
Other:
- moved on the sheet: D1, R2
Changed lines of the file:
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@@
 <attribute name="OCTOPART_URL" value="https://octopart.com/vlms1300-gs08-vishay-21709201?r=sp&amp;s=_gcP4_q8T1SC6PJQPTQ9yA"/>
 </part>
-<part name="X1" library="Hexabitz" deviceset="XTALL_CSTCE8M00G52" device="" package3d_urn="urn:adsk.eagle:package:20064680/2" value="XTALL_CSTCE8M00G52"/>
+<part name="X1" library="HEXABITZ_RCLS" library_urn="urn:adsk.eagle:library:20064561" deviceset="XTALL_CSTCE8M00G52" device="" package3d_urn="urn:adsk.eagle:package:20410717/1" value="XTALL_CSTCE8M00G52"/>
 <part name="GND1" library="supply1" library_urn="urn:adsk.eagle:library:371" deviceset="GND" device=""/>
 <part name="SUPPLY14" library="supply2" library_urn="urn:adsk.eagle:library:372" deviceset="VDD" device=""/>
@@
 <attribute name="MPN" value="C1608X7R1H104K080AA"/>
 </part>
-<part name="TVS1" library="HEXABITZ_RCLS" library_urn="urn:adsk.eagle:library:20064561" deviceset="SMBJ30CA" device="" package3d_urn="urn:adsk.eagle:package:19666516/2"/>
-<part name="TVS2" library="HEXABITZ_RCLS" library_urn="urn:adsk.eagle:library:20064561" deviceset="SMBJ30CA" device="" package3d_urn="urn:adsk.eagle:package:19666516/2"/>
+<part name="TVS1" library="HEXABITZ_RCLS" library_urn="urn:adsk.eagle:library:20064561" deviceset="SMBJ30CA" device="" package3d_urn="urn:adsk.eagle:package:19666516/3"/>
+<part name="TVS2" library="HEXABITZ_RCLS" library_urn="urn:adsk.eagle:library:20064561" deviceset="SMBJ30CA" device="" package3d_urn="urn:adsk.eagle:package:19666516/3"/>
 <part name="D2" library="HEXABITZ_RCLS" library_urn="urn:adsk.eagle:library:20064561" deviceset="DIOD-SOD-123" device="" package3d_urn="urn:adsk.eagle:package:19666494/2"/>
 <part name="D3" library="HEXABITZ_RCLS" library_urn="urn:adsk.eagle:library:20064561" deviceset="DIOD-SOD-123" device="" package3d_urn="urn:adsk.eagle:package:19666494/2"/>
@@
 </plain>
 <instances>
-<instance part="D1" gate="G$1" x="234.315" y="113.665" smashed="yes" rot="R180">
-<attribute name="NAME" x="231.648" y="110.109" size="1.778" layer="95"/>
-<attribute name="VALUE" x="238.252" y="117.475" size="1.778" layer="96" rot="R180"/>
+<instance part="D1" gate="G$1" x="121.285" y="107.315" smashed="yes" rot="R90">
+<attribute name="NAME" x="117.729" y="109.982" size="1.778" layer="95" rot="R270"/>
+<attribute name="VALUE" x="125.095" y="103.378" size="1.778" layer="96" rot="R90"/>
 </instance>
 <instance part="X1" gate="G$1" x="111.125" y="154.305" smashed="yes" rot="MR90">
@@
 <attribute name="VALUE" x="125.73" y="158.75" size="1.778" layer="96" rot="MR0"/>
 </instance>
-<instance part="GND1" gate="1" x="245.11" y="111.125" smashed="yes">
-<attribute name="VALUE" x="242.57" y="108.585" size="1.778" layer="96"/>
+<instance part="GND1" gate="1" x="121.285" y="100.965" smashed="yes">
+<attribute name="VALUE" x="118.745" y="98.425" size="1.778" layer="96"/>
 </instance>
 <instance part="SUPPLY14" gate="G$1" x="226.06" y="128.905" smashed="yes">
@@
 <attribute name="VALUE" x="249.047" y="127" size="1.778" layer="96" rot="R90"/>
 </instance>
-<instance part="R2" gate="G$1" x="224.155" y="113.665" smashed="yes">
-<attribute name="NAME" x="222.885" y="110.0836" size="1.778" layer="95"/>
-<attribute name="VALUE" x="221.615" y="115.443" size="1.778" layer="96"/>
+<instance part="R2" gate="G$1" x="121.285" y="116.205" smashed="yes" rot="R270">
+<attribute name="NAME" x="117.7036" y="117.475" size="1.778" layer="95" rot="R270"/>
+<attribute name="VALUE" x="123.063" y="118.745" size="1.778" layer="96" rot="R270"/>
 </instance>
 <instance part="R1" gate="G$1" x="207.645" y="50.165" smashed="yes">
@@
 <pinref part="GND1" gate="1" pin="GND"/>
 <pinref part="D1" gate="G$1" pin="C"/>
-<wire x1="245.11" y1="113.665" x2="239.395" y2="113.665" width="0.1524" layer="91"/>
+<wire x1="121.285" y1="103.505" x2="121.285" y2="102.235" width="0.1524" layer="91"/>
 </segment>
 <segment>
@@
 <segment>
 <pinref part="GND18" gate="1" pin="GND"/>
-<wire x1="226.06" y1="123.825" x2="217.17" y2="123.825" width="0.1524" layer="91"/>
+<wire x1="226.06" y1="123.825" x2="219.71" y2="123.825" width="0.1524" layer="91"/>
 <pinref part="U1" gate="A" pin="VSS"/>
+<pinref part="U1" gate="A" pin="PA9"/>
+<wire x1="219.71" y1="123.825" x2="217.17" y2="123.825" width="0.1524" layer="91"/>
+<wire x1="217.17" y1="121.285" x2="219.71" y2="121.285" width="0.1524" layer="91"/>
+<wire x1="219.71" y1="121.285" x2="219.71" y2="123.825" width="0.1524" layer="91"/>
+<junction x="219.71" y="123.825"/>
 </segment>
 <segment>
@@
 <segment>
 <pinref part="D1" gate="G$1" pin="A"/>
-<wire x1="231.775" y1="113.665" x2="229.235" y2="113.665" width="0.1524" layer="91"/>
 <pinref part="R2" gate="G$1" pin="2"/>
+<wire x1="121.285" y1="109.855" x2="121.285" y2="111.125" width="0.1524" layer="91"/>
 </segment>
 </net>
@@
 <segment>
 <wire x1="109.855" y1="129.54" x2="109.855" y2="133.35" width="0.1524" layer="91"/>
-<wire x1="146.05" y1="149.225" x2="120.65" y2="149.225" width="0.1524" layer="91"/>
-<wire x1="120.65" y1="149.225" x2="120.65" y2="133.35" width="0.1524" layer="91"/>
-<wire x1="120.65" y1="133.35" x2="109.855" y2="133.35" width="0.1524" layer="91"/>
+<wire x1="146.05" y1="149.225" x2="114.935" y2="149.225" width="0.1524" layer="91"/>
+<wire x1="114.935" y1="149.225" x2="114.935" y2="133.35" width="0.1524" layer="91"/>
+<wire x1="114.935" y1="133.35" x2="109.855" y2="133.35" width="0.1524" layer="91"/>
 <pinref part="R" gate="G$1" pin="1"/>
 <wire x1="101.6" y1="133.35" x2="109.855" y2="133.35" width="0.1524" layer="91"/>
@@
 </segment>
 </net>
-<net name="USART6_TX" class="0">
-<segment>
-<wire x1="129.54" y1="136.525" x2="146.05" y2="136.525" width="0.1524" layer="91"/>
-<pinref part="U1" gate="A" pin="PA4"/>
-<label x="129.54" y="136.525" size="1.778" layer="95"/>
-</segment>
-</net>
-<net name="USART6_RX" class="0">
-<segment>
-<wire x1="129.54" y1="133.985" x2="146.05" y2="133.985" width="0.1524" layer="91"/>
-<pinref part="U1" gate="A" pin="PA5"/>
-<label x="129.54" y="133.985" size="1.778" layer="95"/>
-</segment>
-</net>
 <net name="USART4_TX" class="0">
 <segment>
@@
 <pinref part="P1" gate="G$1" pin="SD1"/>
 <label x="63.5" y="137.16" size="1.778" layer="95"/>
-</segment>
-</net>
-<net name="N$15" class="0">
-<segment>
-<pinref part="U1" gate="A" pin="PB14"/>
-<pinref part="R2" gate="G$1" pin="1"/>
-<wire x1="217.17" y1="113.665" x2="219.075" y2="113.665" width="0.1524" layer="91"/>
 </segment>
 </net>
@@
 <net name="M_SIG" class="0">
 <segment>
-<label x="117.475" y="100.33" size="1.778" layer="95" rot="R180" xref="yes"/>
-<wire x1="130.175" y1="100.33" x2="117.475" y2="100.33" width="0.1524" layer="91"/>
+<label x="135.255" y="136.525" size="1.778" layer="95" rot="R180" xref="yes"/>
+<wire x1="146.05" y1="136.525" x2="135.255" y2="136.525" width="0.1524" layer="91"/>
+<pinref part="U1" gate="A" pin="PA4"/>
 </segment>
 </net>
+<net name="USART3_TX" class="0">
+<segment>
+<wire x1="129.54" y1="118.745" x2="146.05" y2="118.745" width="0.1524" layer="91"/>
+<pinref part="U1" gate="A" pin="PB10"/>
+<label x="129.54" y="118.745" size="1.778" layer="95"/>
+</segment>
+<segment>
+<wire x1="60.96" y1="162.56" x2="77.47" y2="162.56" width="0.1524" layer="91"/>
+<pinref part="P1" gate="G$1" pin="SU3"/>
+<label x="63.5" y="162.56" size="1.778" layer="95"/>
+</segment>
+</net>
+<net name="USART3_RX" class="0">
+<segment>
+<wire x1="129.54" y1="116.205" x2="146.05" y2="116.205" width="0.1524" layer="91"/>
+<pinref part="U1" gate="A" pin="PB11"/>
+<label x="129.54" y="116.205" size="1.778" layer="95"/>
+</segment>
+<segment>
+<wire x1="60.96" y1="127" x2="77.47" y2="127" width="0.1524" layer="91"/>
+<pinref part="P1" gate="G$1" pin="SD3"/>
+<label x="63.5" y="127" size="1.778" layer="95"/>
+</segment>
+</net>
+<net name="N$4" class="0">
+<segment>
+<pinref part="R2" gate="G$1" pin="1"/>
+<wire x1="121.285" y1="121.285" x2="146.05" y2="121.285" width="0.1524" layer="91"/>
+<pinref part="U1" gate="A" pin="PB2"/>
+</segment>
+</net>

Commit message: -All done
Parts:
- R4: value 5K -> 4.99K
- renumbered R to RESET
Other:
- note added: "VREF = 3 Volt"
- note added: "Vo = Gain * Vin + VREF/2 Gain = (0.1) * (1 + R4/R5)"
- note removed: "Vo = (0.1) * (1 + 5/10) Vin"
Changed lines of the file:
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@@
 <attribute name="OCTOPART_URL" value="https://octopart.com/vlms1300-gs08-vishay-21709201?r=sp&amp;s=_gcP4_q8T1SC6PJQPTQ9yA"/>
 </part>
-<part name="X1" library="HEXABITZ_RCLS" library_urn="urn:adsk.eagle:library:20064561" deviceset="XTALL_CSTCE8M00G52" device="" package3d_urn="urn:adsk.eagle:package:20410717/1" value="XTALL_CSTCE8M00G52"/>
+<part name="X1" library="HEXABITZ_RCLS" library_urn="urn:adsk.eagle:library:20064561" deviceset="XTALL_CSTCE8M00G52" device="" package3d_urn="urn:adsk.eagle:package:20410717/3" value="XTALL_CSTCE8M00G52"/>
 <part name="GND1" library="supply1" library_urn="urn:adsk.eagle:library:371" deviceset="GND" device=""/>
 <part name="SUPPLY14" library="supply2" library_urn="urn:adsk.eagle:library:372" deviceset="VDD" device=""/>
@@
 <part name="GND8" library="supply1" library_urn="urn:adsk.eagle:library:371" deviceset="GND" device=""/>
 <part name="GND10" library="supply1" library_urn="urn:adsk.eagle:library:371" deviceset="GND" device=""/>
-<part name="R" library="HEXABITZ_USER_INTERFACE_PARTS" library_urn="urn:adsk.eagle:library:20064563" deviceset="PINHD-1X1" device="" package3d_urn="urn:adsk.eagle:package:22485/2" value="R"/>
+<part name="RESET" library="HEXABITZ_USER_INTERFACE_PARTS" library_urn="urn:adsk.eagle:library:20064563" deviceset="PINHD-1X1" device="" package3d_urn="urn:adsk.eagle:package:22485/2" value="R"/>
 <part name="GND9" library="supply1" library_urn="urn:adsk.eagle:library:371" deviceset="GND" device=""/>
 <part name="GND18" library="supply1" library_urn="urn:adsk.eagle:library:371" deviceset="GND" device=""/>
@@
 <part name="U2" library="HEXABITZ_ICs" library_urn="urn:adsk.eagle:library:20064554" deviceset="AD628ARZ" device="" package3d_urn="urn:adsk.eagle:package:19881610/4"/>
 <part name="C8" library="HEXABITZ_RCLS" library_urn="urn:adsk.eagle:library:20064561" deviceset="C-0603" device="" package3d_urn="urn:adsk.eagle:package:19666468/3" value="15nF"/>
-<part name="R4" library="HEXABITZ_RCLS" library_urn="urn:adsk.eagle:library:20064561" deviceset="R-0603" device="" package3d_urn="urn:adsk.eagle:package:1435818/6" value="5K"/>
+<part name="R4" library="HEXABITZ_RCLS" library_urn="urn:adsk.eagle:library:20064561" deviceset="R-0603" device="" package3d_urn="urn:adsk.eagle:package:1435818/6" value="4.99K"/>
 <part name="P+3" library="HEXABITZ_CONNECTION_PARTS" library_urn="urn:adsk.eagle:library:20064553" deviceset="VREF/2" device=""/>
 <part name="P+4" library="HEXABITZ_CONNECTION_PARTS" library_urn="urn:adsk.eagle:library:20064553" deviceset="+VS" device=""/>
@@
 <attribute name="MPN" value="C1608X7R1H104K080AA"/>
 </part>
-<part name="TVS1" library="HEXABITZ_RCLS" library_urn="urn:adsk.eagle:library:20064561" deviceset="SMBJ30CA" device="" package3d_urn="urn:adsk.eagle:package:19666516/3"/>
-<part name="TVS2" library="HEXABITZ_RCLS" library_urn="urn:adsk.eagle:library:20064561" deviceset="SMBJ30CA" device="" package3d_urn="urn:adsk.eagle:package:19666516/3"/>
-<part name="D2" library="HEXABITZ_RCLS" library_urn="urn:adsk.eagle:library:20064561" deviceset="DIOD-SOD-123" device="" package3d_urn="urn:adsk.eagle:package:19666494/2"/>
-<part name="D3" library="HEXABITZ_RCLS" library_urn="urn:adsk.eagle:library:20064561" deviceset="DIOD-SOD-123" device="" package3d_urn="urn:adsk.eagle:package:19666494/2"/>
-<part name="SWD" library="HEXABITZ_CONNECTION_PARTS" library_urn="urn:adsk.eagle:library:20064553" deviceset="PINHD-1X3" device="SWD" package3d_urn="urn:adsk.eagle:package:42172676/1"/>
+<part name="TVS1" library="HEXABITZ_RCLS" library_urn="urn:adsk.eagle:library:20064561" deviceset="SMBJ30CA" device="" package3d_urn="urn:adsk.eagle:package:19666516/4"/>
+<part name="TVS2" library="HEXABITZ_RCLS" library_urn="urn:adsk.eagle:library:20064561" deviceset="SMBJ30CA" device="" package3d_urn="urn:adsk.eagle:package:19666516/4"/>
+<part name="D2" library="HEXABITZ_RCLS" library_urn="urn:adsk.eagle:library:20064561" deviceset="DIOD-SOD-123" device="" package3d_urn="urn:adsk.eagle:package:19666494/3"/>
+<part name="D3" library="HEXABITZ_RCLS" library_urn="urn:adsk.eagle:library:20064561" deviceset="DIOD-SOD-123" device="" package3d_urn="urn:adsk.eagle:package:19666494/3"/>
+<part name="SWD" library="HEXABITZ_CONNECTION_PARTS" library_urn="urn:adsk.eagle:library:20064553" deviceset="PINHD-1X3" device="SWD" package3d_urn="urn:adsk.eagle:package:42172676/2"/>
 <part name="P+8" library="HEXABITZ_CONNECTION_PARTS" library_urn="urn:adsk.eagle:library:20064553" deviceset="+VS" device=""/>
 <part name="P-3" library="HEXABITZ_CONNECTION_PARTS" library_urn="urn:adsk.eagle:library:20064553" deviceset="-VS" device=""/>
@@
 <part name="SUPPLY19" library="HEXABITZ_CONNECTION_PARTS" library_urn="urn:adsk.eagle:library:20064553" deviceset="VSSA" device=""/>
 <part name="P1" library="hexabitz_connectors" library_urn="urn:adsk.eagle:library:20064578" deviceset="HEXABIT_?_NO_P6_P7_P12" device="17.32" package3d_urn="urn:adsk.eagle:package:20064634/2"/>
-<part name="J1" library="HEXABITZ_CONNECTION_PARTS" library_urn="urn:adsk.eagle:library:20064553" deviceset="1984646" device="" package3d_urn="urn:adsk.eagle:package:42202473/1"/>
+<part name="J1" library="HEXABITZ_CONNECTION_PARTS" library_urn="urn:adsk.eagle:library:20064553" deviceset="1984646" device="" package3d_urn="urn:adsk.eagle:package:42202473/2"/>
 </parts>
 <sheets>
@@
 <attribute name="VALUE" x="103.505" y="145.415" size="1.778" layer="96" rot="MR0"/>
 </instance>
-<instance part="R" gate="G$1" x="99.06" y="133.35" smashed="yes" rot="R180">
-<attribute name="NAME" x="100.33" y="137.16" size="1.778" layer="95"/>
+<instance part="RESET" gate="G$1" x="99.06" y="133.35" smashed="yes" rot="R180">
+<attribute name="NAME" x="97.155" y="137.16" size="1.778" layer="95"/>
 </instance>
 <instance part="GND9" gate="1" x="220.98" y="172.085" smashed="yes" rot="MR270">
@@
 <wire x1="114.935" y1="149.225" x2="114.935" y2="133.35" width="0.1524" layer="91"/>
 <wire x1="114.935" y1="133.35" x2="109.855" y2="133.35" width="0.1524" layer="91"/>
-<pinref part="R" gate="G$1" pin="1"/>
+<pinref part="RESET" gate="G$1" pin="1"/>
 <wire x1="101.6" y1="133.35" x2="109.855" y2="133.35" width="0.1524" layer="91"/>
 <junction x="109.855" y="133.35"/>
@@
 <wire x1="90.805" y1="85.725" x2="90.805" y2="94.615" width="0.1524" layer="90"/>
 <wire x1="90.805" y1="94.615" x2="58.42" y2="94.615" width="0.1524" layer="90"/>
-<text x="207.01" y="84.455" size="2.54" layer="89" font="vector" ratio="11" distance="45">Vo = (0.1) * (1 + 5/10) Vin</text>
-<wire x1="206.375" y1="89.535" x2="206.375" y2="83.185" width="0.1524" layer="90"/>
-<wire x1="206.375" y1="83.185" x2="253.365" y2="83.185" width="0.1524" layer="90"/>
-<wire x1="253.365" y1="83.185" x2="253.365" y2="89.535" width="0.1524" layer="90"/>
-<wire x1="253.365" y1="89.535" x2="206.375" y2="89.535" width="0.1524" layer="90"/>
+<text x="207.01" y="84.455" size="2.54" layer="89" font="vector" ratio="11" distance="45">Vo = Gain * Vin + VREF/2
+Gain = (0.1) * (1 + R4/R5)</text>
+<wire x1="206.375" y1="91.44" x2="206.375" y2="83.185" width="0.1524" layer="90"/>
+<wire x1="206.375" y1="83.185" x2="250.19" y2="83.185" width="0.1524" layer="90"/>
+<wire x1="250.19" y1="83.185" x2="250.19" y2="91.44" width="0.1524" layer="90"/>
+<wire x1="250.19" y1="91.44" x2="206.375" y2="91.44" width="0.1524" layer="90"/>
 <text x="219.71" y="136.525" size="3.81" layer="101" ratio="31">U2 Coupling</text>
+<text x="142.875" y="200.66" size="2.54" layer="89" font="vector" ratio="11" distance="46">VREF = 3 Volt</text>
+<wire x1="142.24" y1="204.47" x2="142.24" y2="199.39" width="0.1524" layer="90"/>
+<wire x1="142.24" y1="199.39" x2="165.735" y2="199.39" width="0.1524" layer="90"/>
+<wire x1="165.735" y1="199.39" x2="165.735" y2="204.47" width="0.1524" layer="90"/>
+<wire x1="165.735" y1="204.47" x2="142.24" y2="204.47" width="0.1524" layer="90"/>
 </plain>
 <instances>
