File: H12R00/Design/H12R00.brd (EAGLE design)
At the start: 34.6 x 30 mm, 42 parts, among them J1 1984646, P1 HEXABIT_17.32_NO_P6_P7_P12, U1 STM32G0B1CEU6N, U2 AD628ARZ, U3 TEXAS_INSTRUMENTS_REF2033AIDD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, X1 XTALL_CSTCE8M00G52

Commit message: -After wiring
Parts:
- X1: device Hexabitz:XTALL_CSTCE8M00G52 -> HEXABITZ_RCLS:XTALL_CSTCE8M00G52
- moved R2 218.4 mm to (5.71, 7.30), turned to 270 degrees
- moved D1 216.4 mm to (5.24, 5.71), turned to 0 degrees
- moved SWD 216.1 mm to (-5.08, 6.03)
- moved R 208.4 mm to (5.24, 9.84)
- moved R1 196.2 mm to (4.60, 16.4), turned to 270 degrees
- moved R3 190.9 mm to (-0.58, 8.95), flipped to the top
- moved C3 187.4 mm to (-2.70, 16.5), turned to 180 degrees
- moved X1 187.3 mm to (1.27, 16.2)
- moved C7 186.9 mm to (0.32, 4.13)
- moved C10 186.8 mm to (3.17, 21.1)
- moved C11 186.8 mm to (-3.33, 21.1)
- moved C18 186.8 mm to (-4.76, 15.9)
- moved C19 186.8 mm to (5.24, 19.4)
- moved C20 186.8 mm to (-5.56, 19.4)
- moved C6 186.8 mm to (0.32, 5.24)
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Connections:
- removed net N$15: R2.1, U1.26
- removed net USART6_RX: U1.16
- removed net USART6_TX: U1.15
- new net N$4: R2.1, U1.21
- new net USART3_RX: P1.PAD_PD3, U1.23
- new net USART3_TX: P1.PAD_PU3, U1.22
- net GND: now also U1.29
- net M_SIG: now also U1.15
Routing:
- net USART4_TX: track 0.00 -> 19.0 mm, vias 0 -> 1
- net USART1_TX: track 0.00 -> 18.9 mm, vias 0 -> 1
- net USART1_RX: track 0.00 -> 18.3 mm
- net USART4_RX: track 0.00 -> 17.3 mm
- net GND: track 0.00 -> 15.3 mm, vias 0 -> 16
- net VDDA: track 0.00 -> 12.0 mm, vias 0 -> 1
- net USART5_RX: track 0.00 -> 11.6 mm
- net USART5_TX: track 0.00 -> 11.4 mm, vias 0 -> 1
- net USART3_TX: track 0.00 -> 11.1 mm, vias 0 -> 1
- net USART2_TX: track 0.00 -> 10.7 mm, vias 0 -> 1
- net USART2_RX: track 0.00 -> 10.6 mm
- net CLK: track 0.00 -> 9.92 mm
- net USART3_RX: track 0.00 -> 9.30 mm
- net IN+: track 0.00 -> 8.55 mm
- net IN-: track 0.00 -> 8.22 mm
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- added copper zone on layer 1, net +VS
- added copper zone on layer 1, net -VS
- added copper zone on layer 1, net CFILT
- added copper zone on layer 1, net GND
- added copper zone on layer 16, net GND
- added copper zone on layer 1, net VDD
- added copper zone on layer 1, net VDDA
- added copper zone on layer 1, net VREF
- added copper zone on layer 1, net VREF/2
- added copper zone on layer 1, net VSSA
- added copper zone on layer 16, net VSSA
Other:
- board text added: "AIN+"
- board text added: "AIN-"
- board text added: "AIN_MAX=±10V"
- board text added: "P2*"
- board text added: "P3"
- board text added: "VS+"
- board text added: "VS-"
- board text added: "VS_MAX=±15V"
- board text removed: "*P2"

Commit message: -All done
Parts:
- R4: value 5K -> 4.99K
- moved C2 1.57 mm to (-1.59, 16.5), turned to 90 degrees
- moved C5 1.28 mm to (-5.56, 13.5)
- moved C4 1.14 mm to (-4.45, 13.5)
- moved R1 0.32 mm to (4.92, 16.4)
- turned C3 to 90 degrees
- renumbered R to RESET
Routing:
- net GND: track 15.3 -> 16.8 mm
- net VREF: track 8.04 -> 6.75 mm
- net VSSA: track 3.69 -> 4.82 mm, vias 16 -> 17
- net -VS: track 6.40 -> 5.56 mm
- net VDDA: track 12.0 -> 11.2 mm
